Commit message: Update myrobot.xacro

File: urdf/myrobot.xacro (robot description, xacro)
@@ -32,11 +32,4 @@
     <child link="$(arg base_frame)" />
   </joint>
-<!--
-  <joint name="camera_joint" type="fixed">
-    <origin xyz="0.26 0 0" rpy="0 0 0" />
-    <parent link="chassis"/>
-    <child link="camera" />
-    <axis xyz="0 1 0"/>
-  </joint>-->
   <joint name="hokuyo_joint" type="fixed">
     <origin xyz="0 0 0.2" rpy="0 0 0" />
@@ -66,15 +59,7 @@
      <child link="camera_depth_frame" />
   </joint>
-<!--
-  <joint name="left_camera_frame_joint" type="fixed">
-     <origin xyz="0 0 0.45" rpy="0 0 0" />
-     <parent link="$(arg base_frame)" />
-     <child link="left_camera_frame" />
-  </joint>
--->
-<!--
-<link name="camera">
-    <inertial>
-      <mass value="0.1"/>
+  <link name="hokuyo">
+    <inertial>
+      <mass value="1e-5"/>
       <origin xyz="0 0 0" rpy="0 0 0"/>
       <inertia
@@ -87,17 +72,17 @@
       <origin xyz="0 0 0" rpy="0 0 0"/>
       <geometry>
-        <box size="0.05 0.05 0.05"/>
-      </geometry>
-    </collision>
-    <visual>
-      <origin xyz="0 0 0" rpy="0 0 0"/>
-      <geometry>
-        <box size="0.05 0.05 0.05"/>
-      </geometry>
-    </visual>
-  </link>-->
-  <link name="hokuyo">
-    <inertial>
-      <mass value="1e-5"/>
+        <box size="0.1 0.1 0.1"/>
+      </geometry>
+    </collision>
+    <visual>
+      <origin xyz="0.1 0 0" rpy="0 0 0"/>
+      <geometry>
+        <mesh filename="package://project/meshes/hokuyo.dae"/>
+      </geometry>
+    </visual>
+  </link>
+  <link name="camera_depth_frame">
+    <inertial>
+      <mass value="0.1"/>
       <origin xyz="0 0 0" rpy="0 0 0"/>
       <inertia
@@ -110,27 +95,4 @@
       <origin xyz="0 0 0" rpy="0 0 0"/>
       <geometry>
-        <box size="0.1 0.1 0.1"/>
-      </geometry>
-    </collision>
-    <visual>
-      <origin xyz="0.1 0 0" rpy="0 0 0"/>
-      <geometry>
-        <mesh filename="package://project/meshes/hokuyo.dae"/>
-      </geometry>
-    </visual>
-  </link>
-  <link name="camera_depth_frame">
-    <inertial>
-      <mass value="0.1"/>
-      <origin xyz="0 0 0" rpy="0 0 0"/>
-      <inertia
-        ixx="1e-6" ixy="0.0" ixz="0.0"
-        iyy="1e-6" iyz="0.0"
-        izz="1e-6"
-      />
-    </inertial>
-    <collision>
-      <origin xyz="0 0 0" rpy="0 0 0"/>
-      <geometry>
         <box size="0.05 0.05 0.05"/>
       </geometry>
@@ -237,28 +199,3 @@
     </visual>
   </link>
-<!--
-  <link name="left_camera_frame">
-    <inertial>
-      <mass value="0.1"/>
-      <origin xyz="0 0 0" rpy="0 0 0"/>
-      <inertia
-        ixx="1e-6" ixy="0.0" ixz="0.0"
-        iyy="1e-6" iyz="0.0"
-        izz="1e-6"
-      />
-    </inertial>
-    <collision>
-      <origin xyz="0 0 0" rpy="0 0 0"/>
-      <geometry>
-        <box size="0.05 0.05 0.05"/>
-      </geometry>
-    </collision>
-    <visual>
-      <origin xyz="0 0 0" rpy="0 0 0"/>
-      <geometry>
-        <mesh filename="package://project/meshes/zed.stl"/>
-      </geometry>
-    </visual>
-  </link>
--->
 </robot>

Commit message: Update myrobot.xacro

File: urdf/myrobot.xacro (robot description, xacro)
@@ -10,8 +10,4 @@
     <material>Gazebo/Green</material>
   </gazebo>
-<!--
-  <gazebo reference="camera">
-    <material>Gazebo/Red</material>
-  </gazebo>-->
   <gazebo reference="$(arg base_frame)">
     <material>Gazebo/Blue</material>
